File: breakout-lrtb-g6tg_light.brd (EAGLE design)
At the start: 22.9 x 12.7 mm, 3 parts

Commit message: nochmal anders
Parts:
- turned LED1 to 270 degrees
Connections:
- net N$7: now also JP2.3; no longer JP2.2
- net N$9: now also JP2.2; no longer JP2.3
Routing:
- net N$9: track 11.5 -> 21.1 mm, vias 0 -> 2
- net N$5: track 6.31 -> 14.2 mm
- net N$6: track 14.1 -> 6.24 mm
- net N$8: track 14.4 -> 8.42 mm
- net N$7: track 7.36 -> 6.24 mm
Changed lines of the file:
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@@
 <setting verticaltext="up"/>
 </settings>
-<grid distance="25" unitdist="mil" unit="mil" style="lines" multiple="4" display="yes" altdistance="25" altunitdist="mil" altunit="mil"/>
+<grid distance="25" unitdist="mil" unit="mil" style="lines" multiple="1" display="yes" altdistance="25" altunitdist="mil" altunit="mil"/>
 <layers>
 <layer number="1" name="Top" color="4" fill="1" visible="yes" active="yes"/>
@@
 <wire x1="22.86" y1="12.7" x2="0" y2="12.7" width="0" layer="20"/>
 <wire x1="0" y1="12.7" x2="0" y2="0" width="0" layer="20"/>
-<rectangle x1="12.7" y1="8.89" x2="13.97" y2="11.43" layer="42"/>
+<rectangle x1="13.97" y1="5.715" x2="15.875" y2="6.985" layer="42"/>
+<rectangle x1="10.795" y1="1.905" x2="12.065" y2="5.715" layer="42"/>
+<rectangle x1="5.715" y1="10.795" x2="6.35" y2="11.43" layer="42"/>
+<rectangle x1="0" y1="4.445" x2="1.27" y2="8.255" layer="42"/>
+<rectangle x1="21.59" y1="4.445" x2="22.86" y2="8.255" layer="42"/>
 </plain>
 <attributes>
@@
 </autorouter>
 <elements>
-<element name="LED1" library="led" package="LRTB_G6SG" value="LRTB_G6SG" x="11.43" y="6.35" rot="MR180"/>
+<element name="LED1" library="led" package="LRTB_G6SG" value="LRTB_G6SG" x="11.43" y="6.35" rot="MR270"/>
 <element name="JP2" library="pinhead" package="1X03" value="" x="2.54" y="6.35" rot="R90"/>
 <element name="JP3" library="pinhead" package="1X03" value="" x="20.32" y="6.35" rot="R270"/>
@@
 <contactref element="JP3" pad="2"/>
 <contactref element="LED1" pad="3"/>
-<wire x1="14.08" y1="9.05" x2="16.78" y2="6.35" width="0.6096" layer="16"/>
-<wire x1="16.78" y1="6.35" x2="20.32" y2="6.35" width="0.6096" layer="16"/>
+<wire x1="20.32" y1="6.35" x2="16.78" y2="6.35" width="0.6096" layer="16"/>
+<wire x1="16.78" y1="6.35" x2="14.13" y2="3.7" width="0.6096" layer="16"/>
 </signal>
 <signal name="N$5">
 <contactref element="JP3" pad="3"/>
 <contactref element="LED1" pad="4"/>
-<wire x1="14.08" y1="3.65" x2="14.24" y2="3.81" width="0.6096" layer="16"/>
-<wire x1="14.24" y1="3.81" x2="20.32" y2="3.81" width="0.6096" layer="16"/>
+<wire x1="8.73" y1="3.7" x2="11.795" y2="0.635" width="0.6096" layer="16"/>
+<wire x1="11.795" y1="0.635" x2="16.51" y2="0.635" width="0.6096" layer="16"/>
+<wire x1="16.51" y1="0.635" x2="19.685" y2="3.81" width="0.6096" layer="16"/>
+<wire x1="19.685" y1="3.81" x2="20.32" y2="3.81" width="0.6096" layer="16"/>
 </signal>
 <signal name="N$6">
 <contactref element="JP3" pad="1"/>
 <contactref element="LED1" pad="1"/>
-<wire x1="8.78" y1="9.05" x2="11.795" y2="12.065" width="0.6096" layer="16"/>
-<wire x1="11.795" y1="12.065" x2="16.51" y2="12.065" width="0.6096" layer="16"/>
-<wire x1="16.51" y1="12.065" x2="19.685" y2="8.89" width="0.6096" layer="16"/>
-<wire x1="19.685" y1="8.89" x2="20.32" y2="8.89" width="0.6096" layer="16"/>
+<wire x1="14.13" y1="9" x2="14.24" y2="8.89" width="0.6096" layer="16"/>
+<wire x1="14.24" y1="8.89" x2="20.32" y2="8.89" width="0.6096" layer="16"/>
 </signal>
 <signal name="N$7">
-<contactref element="JP2" pad="2"/>
 <contactref element="LED1" pad="6"/>
-<wire x1="8.78" y1="3.65" x2="5.875" y2="3.65" width="0.6096" layer="16"/>
-<wire x1="5.875" y1="3.65" x2="3.175" y2="6.35" width="0.6096" layer="16"/>
-<wire x1="3.175" y1="6.35" x2="2.54" y2="6.35" width="0.6096" layer="16"/>
+<contactref element="JP2" pad="3"/>
+<wire x1="8.73" y1="9" x2="8.62" y2="8.89" width="0.6096" layer="16"/>
+<wire x1="8.62" y1="8.89" x2="2.54" y2="8.89" width="0.6096" layer="16"/>
 </signal>
 <signal name="N$8">
 <contactref element="JP2" pad="1"/>
 <contactref element="LED1" pad="5"/>
-<wire x1="11.43" y1="4.825" x2="11.43" y2="0.635" width="0.6096" layer="16"/>
-<wire x1="11.43" y1="0.635" x2="6.35" y2="0.635" width="0.6096" layer="16"/>
-<wire x1="6.35" y1="0.635" x2="3.175" y2="3.81" width="0.6096" layer="16"/>
-<wire x1="3.175" y1="3.81" x2="2.54" y2="3.81" width="0.6096" layer="16"/>
+<wire x1="9.905" y1="6.35" x2="6.35" y2="6.35" width="0.6096" layer="16"/>
+<wire x1="6.35" y1="6.35" x2="3.81" y2="3.81" width="0.6096" layer="16"/>
+<wire x1="3.81" y1="3.81" x2="2.54" y2="3.81" width="0.6096" layer="16"/>
 </signal>
 <signal name="N$9">
-<contactref element="JP2" pad="3"/>
 <contactref element="LED1" pad="2"/>
-<wire x1="11.43" y1="7.875" x2="11.43" y2="6.35" width="0.6096" layer="16"/>
-<wire x1="11.43" y1="6.35" x2="5.715" y2="6.35" width="0.6096" layer="16"/>
-<wire x1="5.715" y1="6.35" x2="3.175" y2="8.89" width="0.6096" layer="16"/>
-<wire x1="3.175" y1="8.89" x2="2.54" y2="8.89" width="0.6096" layer="16"/>
+<contactref element="JP2" pad="2"/>
+<wire x1="12.955" y1="6.35" x2="11.43" y2="6.35" width="0.6096" layer="16"/>
+<wire x1="11.43" y1="6.35" x2="11.43" y2="12.065" width="0.6096" layer="16"/>
+<wire x1="11.43" y1="12.065" x2="5.08" y2="12.065" width="0.6096" layer="16"/>
+<wire x1="5.08" y1="12.065" x2="5.08" y2="10.16" width="0.6096" layer="16"/>
+<via x="5.08" y="10.16" extent="1-16" drill="0.6" shape="octagon"/>
+<wire x1="5.08" y1="10.16" x2="5.08" y2="7.62" width="0.6096" layer="1"/>
+<via x="5.08" y="7.62" extent="1-16" drill="0.6" shape="octagon"/>
+<wire x1="5.08" y1="7.62" x2="3.81" y2="6.35" width="0.6096" layer="16"/>
+<wire x1="3.81" y1="6.35" x2="2.54" y2="6.35" width="0.6096" layer="16"/>
 </signal>
 <signal name="N$13">
@@
 </polygon>
 </signal>
+<signal name="N$1">
+<via x="5.08" y="7.62" extent="1-16" drill="0.6" shape="octagon"/>
+</signal>
+<signal name="N$2">
+<via x="5.08" y="10.16" extent="1-16" drill="0.6" shape="octagon"/>
+</signal>
 </signals>
