File: breakout-lrtb-g6tg_light.sch (EAGLE design)
At the start: 3 parts

Commit message: nochmal anders
Connections:
- net N$7: now also JP2.3; no longer JP2.2
- net N$9: now also JP2.2; no longer JP2.3
Changed lines of the file:
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@@
 <net name="N$7" class="0">
 <segment>
-<pinref part="JP2" gate="A" pin="2"/>
-<wire x1="40.64" y1="68.58" x2="33.02" y2="68.58" width="0.1524" layer="91"/>
 <pinref part="LED1" gate="-1" pin="C"/>
-<wire x1="33.02" y1="68.58" x2="33.02" y2="58.42" width="0.1524" layer="91"/>
 <wire x1="33.02" y1="58.42" x2="27.94" y2="58.42" width="0.1524" layer="91"/>
+<wire x1="33.02" y1="58.42" x2="33.02" y2="66.04" width="0.1524" layer="91"/>
+<pinref part="JP2" gate="A" pin="3"/>
+<wire x1="33.02" y1="66.04" x2="40.64" y2="66.04" width="0.1524" layer="91"/>
 </segment>
 </net>
@@
 <net name="N$9" class="0">
 <segment>
-<pinref part="JP2" gate="A" pin="3"/>
-<wire x1="40.64" y1="66.04" x2="30.48" y2="66.04" width="0.1524" layer="91"/>
-<wire x1="30.48" y1="66.04" x2="30.48" y2="68.58" width="0.1524" layer="91"/>
 <pinref part="LED1" gate="-2" pin="C"/>
-<wire x1="30.48" y1="68.58" x2="27.94" y2="68.58" width="0.1524" layer="91"/>
+<pinref part="JP2" gate="A" pin="2"/>
+<wire x1="40.64" y1="68.58" x2="27.94" y2="68.58" width="0.1524" layer="91"/>
 </segment>
 </net>
