File: breakout-boards/breakout-ws2812.sch (EAGLE design)
At the start: 7 parts

Commit message: Schönheitskorrekturen
Connections:
- net JDD renamed VDD
- net N$3 renamed VCC
Changed lines of the file:
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@@
 </busses>
 <nets>
-<net name="JDD" class="0">
+<net name="VDD" class="0">
 <segment>
 <pinref part="R1" gate="G$1" pin="2"/>
@@
 </segment>
 </net>
-<net name="N$3" class="0">
+<net name="VCC" class="0">
 <segment>
 <pinref part="R1" gate="G$1" pin="1"/>
@@
 </sheet>
 </sheets>
+<errors>
+</errors>
 </schematic>
 </drawing>
